File: Dual_Wind_Sensor-NANO_noReg.kicad_pcb (KiCad board)
At the start: 4 copper layers, 52.5 x 63.8 mm, 27 parts, among them J1 Screw_Terminal_01x02, J2 Conn_01x05_Pin, J3 Conn_01x05_Pin, J4 Conn_01x03_Pin, J5 Conn_01x05_Pin, U2 HW-613

Commit message: very small change in the PCB.
Other:
- board text added: "V2.0"
Changed lines of the file:
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@@
 			(crossoutdnponfab yes)
 			(subtractmaskfromsilk no)
-			(outputformat 1)
+			(outputformat 4)
 			(mirror no)
 			(drillshape 0)
 			(scaleselection 1)
-			(outputdirectory "Output/")
+			(outputdirectory "Output/Drill/")
 		)
 	)
@@
 		)
 		(embedded_fonts no)
-		(model "${KICAD9_3DMODEL_DIR}/Module.3dshapes/Arduino_Nano_WithMountingHoles.wrl"
-			(offset
-				(xyz 0 0 0)
-			)
-			(scale
-				(xyz 1 1 1)
-			)
-			(rotate
-				(xyz 0 0 0)
-			)
-		)
 		(model "${KICAD9_3DMODEL_DIR}/Arduino.3dshapes/arduino_nano.x3d"
 			(offset
@@
 		(layer "F.SilkS")
 		(effects
+			(font
+				(size 0.8 0.8)
+				(thickness 0.2)
+				(bold yes)
+			)
+			(justify left bottom)
+		)
+	)
+	(gr_text "V2.0"
+		(at 175.6666 85.9976 0)
+		(layer "F.SilkS")
+		(effects
